File: Projet_capteur_pcb/Projet_capteur_pcb.kicad_pcb (KiCad board)
At the start: 2 copper layers, 68.6 x 53.3 mm, 23 parts, among them J1 Power, J2 Digital/PWM, J3 Analog, J4 Digital/PWM

Commit message: model 3D
Parts:
- removed R2: R, Resistor_THT:R_Axial_DIN0207_L6.3mm_D2.5mm_P10.16mm_Horizontal
- moved potD1 37.4 mm to (119.5, 61.5)
- moved Encodeur1 26.7 mm to (147.1, 55.5)
- moved EcranOled1 23.0 mm to (133.2, 55.5)
- moved Bluetooth1 19.4 mm to (159.5, 58.0), turned to -90 degrees
- moved C4 3.64 mm to (124.0, 75.5)
- moved R3 3.14 mm to (136.5, 74.7)
- moved C1 3.04 mm to (148.0, 68.0)
Routing:
- net GND: track 128.9 -> 0.00 mm
- net +5V: track 117.1 -> 0.00 mm
- net SDA: track 101.1 -> 0.00 mm
- net SCL: track 98.7 -> 0.00 mm
- net Net-(AOP1-+IN): track 62.5 -> 0.00 mm
- net Net-(AOP1-OUT): track 51.4 -> 0.00 mm
- net CLK: track 47.2 -> 0.00 mm
- net DT: track 39.4 -> 0.00 mm
- net adc: track 37.8 -> 0.00 mm
- net Net-(AOP1--IN): track 36.7 -> 0.00 mm
- net SW: track 32.8 -> 0.00 mm
- net TxD: track 22.3 -> 0.00 mm
- net Rxd: track 22.3 -> 0.00 mm
- net Net-(C6-OUT): track 16.7 -> 0.00 mm
